Commit message: fix pose of camera frame to pitch link

File: models/iris_with_gimbal_urdf/model.urdf (robot description, URDF)
Before this commit: robot iris_with_gimbal, 11 links, 10 joints
Joints:
- joint camera_optical_joint: origin xyz=0 0 0 rpy=-1.5707963 -1.5707963 0 -> xyz=0 0 0.02 rpy=-1.5707963 -1.5707963 0

Commit message: fix yolo frame and camera frame orientation

File: models/iris_with_gimbal_urdf/model.urdf (robot description, URDF)
Before this commit: robot iris_with_gimbal, 11 links, 10 joints
Links:
- removed link camera_optical_frame
- removed link rotor_0
- removed link rotor_1
- removed link rotor_2
- removed link rotor_3
- added link camera_link
- added link yolo_link
- link base_link: mass 1.5 -> None; geometry visual cylinder length=0.17 radius=0.005; visual cylinder length=0.17 radius=0.005
Joints:
- removed joint camera_optical_joint
- removed joint rotor_0_joint
- removed joint rotor_1_joint
- removed joint rotor_2_joint
- removed joint rotor_3_joint
- added joint camera_joint: type fixed, parent pitch_link, child camera_link, origin xyz=0 0 0.04 rpy=-1.57 -1.57 0
- added joint yolo_joint: type fixed, parent camera_link, child yolo_link, origin xyz=0 0 0 rpy=-1.57 0 -1.57
